Commit message: indigo

File: urdf/ABot.urdf.xacro (robot description, xacro)
@@ -81,5 +81,5 @@
     <child link="right_wheel"/>
     <axis xyz="0 1 0"/>
-    <origin xyz="0.1 -0.15 0.075"/>
+    <origin xyz="0.1 0.15 0.075"/>
   </joint>
   <transmission name="T_base_link_right_wheel">
@@ -119,5 +119,5 @@
     <child link="left_wheel"/>
     <axis xyz="0 1 0"/>
-    <origin xyz="0.1 0.15 0.075"/>
+    <origin xyz="0.1 -0.15 0.075"/>
   </joint>
   <transmission name="T_base_link_left_wheel">
@@ -260,5 +260,5 @@
   </plugin>
 </gazebo>
-  <xacro:include filename="$(find mcl_pi_simulation)/urdf/hokuyo.xacro"/>
+  <xacro:include filename="$(find mcl_pi_gazebo)/urdf/hokuyo.xacro"/>
   <xacro:laser name="base_laser" parent="base_link" xyz="0.225 0 0.2" rpy="0 0 0" meshes="package://gazebo_plugins/test/multi_robot_scenario/meshes/laser"/>
 </robot>

File: urdf/KoBot.urdf.xacro (robot description, xacro)
@@ -81,43 +81,43 @@
     <child link="right_wheel"/>
     <axis xyz="0 1 0"/>
+    <origin xyz="0.1 0.15 0.075"/>
+  </joint>
+  <transmission name="T_base_link_right_wheel">
+    <type>transmission_interface/SimpleTransmission</type>
+    <actuator name="motor_1">
+      <mechanicalReduction>1</mechanicalReduction>
+      <hardwareInterface>hardware_interface/VelocityJointInterface</hardwareInterface>
+    </actuator>
+    <joint name="base_link_right_wheel">
+      <hardwareInterface>hardware_interface/VelocityJointInterface</hardwareInterface>
+    </joint>
+  </transmission>
+  <link name="left_wheel">
+  <inertial>
+    <origin rpy="1.5707963267948966 0 0" xyz="0 0 0" />
+    <mass value="0.1" />
+    <inertia  ixx="0.01" ixy="0.0"  ixz="0.0"  iyy="0.01"  iyz="0.0"  izz="0.01" />
+  </inertial>
+  <visual>
+    <origin rpy="1.5707963267948966 0 0" xyz="0 0 0"/>
+    <geometry>
+      <cylinder length="0.05" radius="0.075"/>
+    </geometry>
+  </visual>
+  <collision>
+    <origin rpy="1.5707963267948966 0 0" xyz="0 0 0"/>
+    <geometry>
+      <cylinder length="0.05" radius="0.075"/>
+    </geometry>
+  </collision>
+  </link>
+  <gazebo reference="left_wheel">
+    <material>Gazebo/Black</material>
+  </gazebo>
+  <joint name="base_link_left_wheel" type="continuous">
+    <parent link="base_link"/>
+    <child link="left_wheel"/>
+    <axis xyz="0 1 0"/>
     <origin xyz="0.1 -0.15 0.075"/>
-  </joint>
-  <transmission name="T_base_link_right_wheel">
-    <type>transmission_interface/SimpleTransmission</type>
-    <actuator name="motor_1">
-      <mechanicalReduction>1</mechanicalReduction>
-      <hardwareInterface>hardware_interface/VelocityJointInterface</hardwareInterface>
-    </actuator>
-    <joint name="base_link_right_wheel">
-      <hardwareInterface>hardware_interface/VelocityJointInterface</hardwareInterface>
-    </joint>
-  </transmission>
-  <link name="left_wheel">
-  <inertial>
-    <origin rpy="1.5707963267948966 0 0" xyz="0 0 0" />
-    <mass value="0.1" />
-    <inertia  ixx="0.01" ixy="0.0"  ixz="0.0"  iyy="0.01"  iyz="0.0"  izz="0.01" />
-  </inertial>
-  <visual>
-    <origin rpy="1.5707963267948966 0 0" xyz="0 0 0"/>
-    <geometry>
-      <cylinder length="0.05" radius="0.075"/>
-    </geometry>
-  </visual>
-  <collision>
-    <origin rpy="1.5707963267948966 0 0" xyz="0 0 0"/>
-    <geometry>
-      <cylinder length="0.05" radius="0.075"/>
-    </geometry>
-  </collision>
-  </link>
-  <gazebo reference="left_wheel">
-    <material>Gazebo/Black</material>
-  </gazebo>
-  <joint name="base_link_left_wheel" type="continuous">
-    <parent link="base_link"/>
-    <child link="left_wheel"/>
-    <axis xyz="0 1 0"/>
-    <origin xyz="0.1 0.15 0.075"/>
   </joint>
   <transmission name="T_base_link_left_wheel">
@@ -270,5 +270,5 @@
         <topicName>/scan</topicName>
         <frameName>/base_laser</frameName> -->
-  <xacro:include filename="$(find mcl_pi_simulation)/urdf/hokuyo.xacro"/>
+  <xacro:include filename="$(find mcl_pi_gazebo)/urdf/hokuyo.xacro"/>
   <xacro:laser name="base_laser" parent="base_link" xyz="0.225 0 0.2" rpy="0 0 0" meshes="package://gazebo_plugins/test/multi_robot_scenario/meshes/laser"/>
 </robot>
